File: Hardware/PCB_Openbook.brd (EAGLE design)
At the start: 170.3 x 111.2 mm, 103 parts, among them IC1 BD5229G-TR, IC4 XC6220A331MR-G, J1 FH34SRJ-24S-0.5SH_99_, J3 QWIIC_RIGHT_ANGLE, J4 112A-TAAR-R03_ATTEND, Q1 20V/4.2A/52mΩ/1.4W, Q2 20V/4.2A/52mΩ/1.4W, Q3 SI1308EDL-T1-GE3, U1 W25Q512JVEIQ, U2 ESP32-C6-WROOM-1-N8, U3 DS3231SN#, U4 MAX17048G+T10

Commit message: Moddified pcb
Parts:
- BOOT_BUTTON, CHANGE_BUTTON, RESET_BUTTON: value BUTTON_CUSYOMV1 -> BUTTON_CUSYOMV1BUTTON
- C1, C10, C1_BAT, C1_BAT1, C1_BAT2, C2, C2_BAT, C4, C4_USB, C5, C5_USB, C6, C7, C8, C9, C_DELAY, EPD_C1, EPD_C10, EPD_C11, EPD_C12, EPD_C2, EPD_C5, EPD_C6, EPD_C7, EPD_C8, EPD_C9: device DeskAssistant v19 v1:ESP32_WROVER_EAGLE-LTSPICE_C0402 -> DeskAssistant v19 v1:EAGLE-LTSPICE_C0402
- D10, D11, D12, D6, D8, D9: value PGB1010603MR -> PGB1010603MRDIODE
- D3, D4, D5: value MBR0530 -> MBR0530DIODE
- J2: value (none) -> SAMACSYS_PARTS_USB4110-GF-A
- MCP73831: value (none) -> ESP32_WROVER_SPARKFUN-IC-POWER_MCP73831
- PFMF.050.1: value (none) -> ESP32C6_VARISTORCN1812
